Commit message: [PycramIntegration] pycram test

File: multiverse/resources/objects/milk_box/urdf/milk_box.urdf (robot description, URDF)
Before this commit: robot milk_box, 1 links, 0 joints
Links:
- link milk_box: geometry collision box size=0.06 0.095 0.2; visual mesh filename=file://milk_box/meshes/obj/milk_box.obj
