Commit message: [FallschoolDemo] Modified apartment to remove all fridge shelves and trays.

File: multiverse/resources/worlds/apartment/urdf/apartment.urdf (robot description, URDF)
Before this commit: robot apartment, 129 links, 128 joints
Links:
- removed link fridge_door_tray1
- removed link fridge_door_tray2
- removed link fridge_drawer1
- removed link fridge_drawer2
- removed link fridge_drawer3
- removed link fridge_drawer4
- removed link fridge_drawer5
- removed link fridge_egg_tray
- removed link fridge_shelf1
- removed link fridge_shelf2
Joints:
- removed joint fridge_door_tray1_joint
- removed joint fridge_door_tray2_joint
- removed joint fridge_drawer1_joint
- removed joint fridge_drawer2_joint
- removed joint fridge_drawer3_joint
- removed joint fridge_drawer4_joint
- removed joint fridge_drawer5_joint
- removed joint fridge_egg_tray_joint
- removed joint fridge_shelf1_joint
- removed joint fridge_shelf2_joint

Commit message: pycram fallschool demo

File: multiverse/resources/worlds/apartment/urdf/apartment.urdf (robot description, URDF)
Before this commit: robot apartment, 119 links, 118 joints
Links:
- link fridge_door1: geometry visual mesh filename=file://../meshes/dae/SM_Fridge_Door_01.dae
- link fridge_door1_handle: geometry visual mesh filename=file://../meshes/dae/SM_Kitchen_Handle.dae
